Commit message: finished Task A.2

File: nuturtle_description/urdf/turtlebot3_burger.urdf.xacro (robot description, xacro)
@@ -44,5 +44,5 @@
       <origin xyz="-0.032 0 0.0" rpy="0 0 0"/>
       <geometry>
-        <mesh filename="package://nuturtle_description/meshes/bases/burger_base.stl" scale="0.001 0.001 0.001"/>
+        <mesh filename="package://nuturtle_description/meshes/burger_base.stl" scale="0.001 0.001 0.001"/>
       </geometry>
       <material name="light_black"/>
@@ -70,5 +70,5 @@
       <origin xyz="0 0 0" rpy="1.57 0 0"/>
       <geometry>
-        <mesh filename="package://nuturtle_description/meshes/wheels/left_tire.stl" scale="0.001 0.001 0.001"/>
+        <mesh filename="package://nuturtle_description/meshes/left_tire.stl" scale="0.001 0.001 0.001"/>
       </geometry>
       <material name="dark"/>
@@ -96,5 +96,5 @@
       <origin xyz="0 0 0" rpy="1.57 0 0"/>
       <geometry>
-        <mesh filename="package://nuturtle_description/meshes/wheels/right_tire.stl" scale="0.001 0.001 0.001"/>
+        <mesh filename="package://nuturtle_description/meshes/right_tire.stl" scale="0.001 0.001 0.001"/>
       </geometry>
       <material name="dark"/>
@@ -145,5 +145,5 @@
       <origin xyz="0 0 0.0" rpy="0 0 0"/>
       <geometry>
-        <mesh filename="package://nuturtle_description/meshes/sensors/lds.stl" scale="0.001 0.001 0.001"/>
+        <mesh filename="package://nuturtle_description/meshes/lds.stl" scale="0.001 0.001 0.001"/>
       </geometry>
       <material name="dark"/>

Commit message: visualizing purple robot, need to add collision_radius conditionals'

File: nuturtle_description/urdf/turtlebot3_burger.urdf.xacro (robot description, xacro)
@@ -3,5 +3,19 @@
   xmlns:xacro="http://ros.org/wiki/xacro">
   <!-- <xacro:include filename="$(find turtlebot3_description)/urdf/common_properties.urdf"/> -->
+ <!-- Modified File from Original file found in the turtlebot3 repo:
+    - Changed file to load in a yaml file for the parameters
+    - Changed pathing parameters for .stl files
+    - Added color launch file argument
+   -->
+<xacro:property name="yaml_file" value="$(find nuturtle_description)/config/diff_params.yaml"/>
+<xacro:property name="props" value="${xacro.load_yaml(yaml_file)['/**']['ros__parameters']}"/>
+<xacro:property name="wheel_radius" value="${props['wheel_radius']}"/>
+<xacro:property name="wheel_track" value="${props['track_width']}"/>
+<xacro:property name="collision_radius" value="${props['collision_radius']}"/>
+<xacro:property name="color" value="purple" />
   <!-- Init colour -->
+  <material name="purple">
+    <color rgba="0.3 0.16 0.52 1.0"/>
+  </material>
   <material name="black">
       <color rgba="0.0 0.0 0.0 1.0"/>
@@ -46,5 +60,5 @@
         <mesh filename="package://nuturtle_description/meshes/burger_base.stl" scale="0.001 0.001 0.001"/>
       </geometry>
-      <material name="light_black"/>
+      <material name="${color}"/>
     </visual>
     <collision>
@@ -63,5 +77,5 @@
     <parent link="base_link"/>
     <child link="wheel_left_link"/>
-    <origin xyz="0.0 0.08 0.023" rpy="-1.57 0 0"/>
+    <origin xyz="0.0 ${wheel_track/2} 0.023" rpy="-1.57 0 0"/>
     <axis xyz="0 0 1"/>
   </joint>
@@ -77,5 +91,5 @@
       <origin xyz="0 0 0" rpy="0 0 0"/>
       <geometry>
-        <cylinder length="0.018" radius="0.033"/>
+        <cylinder length="0.018" radius="${wheel_radius}"/>
       </geometry>
     </collision>
@@ -89,5 +103,5 @@
     <parent link="base_link"/>
     <child link="wheel_right_link"/>
-    <origin xyz="0.0 -0.080 0.023" rpy="-1.57 0 0"/>
+    <origin xyz="0.0 ${-wheel_track/2} 0.023" rpy="-1.57 0 0"/>
     <axis xyz="0 0 1"/>
   </joint>
@@ -103,5 +117,5 @@
       <origin xyz="0 0 0" rpy="0 0 0"/>
       <geometry>
-        <cylinder length="0.018" radius="0.033"/>
+        <cylinder length="0.018" radius="${wheel_radius}"/>
       </geometry>
     </collision>

Commit message: able to change to color of the robot from the launch commandline

File: nuturtle_description/urdf/turtlebot3_burger.urdf.xacro (robot description, xacro)
@@ -13,5 +13,5 @@
 <xacro:property name="wheel_track" value="${props['track_width']}"/>
 <xacro:property name="collision_radius" value="${props['collision_radius']}"/>
-<xacro:property name="color" value="purple" />
+<xacro:property name="color" value="$(arg color)" />
   <!-- Init colour -->
   <material name="purple">

Commit message: progress through Task  A.5 minus frame prefix errors.

File: nuturtle_description/urdf/turtlebot3_burger.urdf.xacro (robot description, xacro)
@@ -62,10 +62,20 @@
       <material name="${color}"/>
     </visual>
-    <collision>
-      <origin xyz="-0.032 0 0.070" rpy="0 0 0"/>
-      <geometry>
-        <box size="0.140 0.140 0.143"/>
-      </geometry>
-    </collision>
+  <xacro:if value="${collision_radius &lt; 0}">
+      <collision>
+        <origin xyz="-0.032 0 0.070" rpy="0 0 0"/>
+        <geometry>
+          <box size="0.140 0.140 0.143"/>
+        </geometry>
+      </collision>
+    </xacro:if>
+    <xacro:unless value="${collision_radius &lt; 0}">
+      <collision>
+        <origin xyz="-0.032 0 0.070" rpy="0 0 0"/>
+        <geometry>
+          <cylinder length="0.143" radius="${collision_radius}"/>
+        </geometry>
+      </collision>
+    </xacro:unless>
     <inertial>
       <origin xyz="0 0 0" rpy="0 0 0"/>
